File: hardware/kicad/USB.kicad_sch (KiCad schematic)
At the start: 33 parts, among them J11 USB_OTG, J13 USB_67298-4090, J14 Conn_02x05_Odd_Even, U13 FSUSB42MUX, U4 TPD4EUSB30, U6 USB2514B_Bi, U7 AP2553W6, Y1 24MHz

Commit message: initial pcb design
Parts:
- removed J11: USB_OTG, CM4IO:USB_Micro-B_EDAC_UCON00686, symbol Connector:USB_OTG
- removed J13: USB_67298-4090, Teapot:MOLEX_USB_67298-4090, symbol Teapot:USB_67298-4090
- removed U4: TPD4EUSB30, Package_SON:USON-10_2.5x1.0mm_P0.5mm, symbol Power_Protection:TPD4EUSB30
- added J5: USB_67298-4090, Teapot:MOLEX_USB_67298-4090, symbol Teapot:USB_67298-4090
- added J7: USB_OTG, Teapot:USB_Micro-B_EDAC_UCON00686, symbol Connector:USB_OTG
- added U4: (no value), symbol Teapot:TPD4EUSB30
Connections:
- net GND: now also J5.4 (GND`), J5.8 (GND), J5.MT1, J5.MT2, J5.MT3, J5.MT4, J7.5 (GND), J7.6 (Shield), U4.3 (GND), U4.8 (GND)
- net HD1_N: now also J5.2 (D-`)
- net HD1_P: now also J5.3 (D+`)
- net HD2_N: now also J5.6 (D-)
- net HD2_P: now also J5.7 (D+)
- net USBD_N: now also J7.2 (D-), U4.4 (D2+), U4.7
- net USBD_P: now also J7.3 (D+), U4.5 (D2-), U4.6
- net USBH_N: now also U13.6 (HSD1-); no longer U13.7 (HSD1+)
- net USBH_P: now also U13.7 (HSD1+); no longer U13.6 (HSD1-)
- net USB_OTG_ID: now also R8.2; no longer R8.1
- net VBUS: now also J5.1 (VBUS`), J5.5 (VBUS)
- new net: J7.1 (VBUS), R8.1
- new net: U4.1 (D1+), U4.10
- new net: U4.2 (D1-), U4.9
Other:
- moved on the sheet: R8
