File: hardware/kicad/data-board/Power.kicad_sch (KiCad schematic)
At the start: 25 parts, among them J1 3.3V LoRaWAN, J2 3.3V SWARM, J4 5V, J6 12V

Commit message: update hole to support solder standoff and decrease pogo pin contact hole size
Parts:
- J1, J2, J4, J6: footprint Connector_Wire:SolderWire-0.5sqmm_1x02_P4.8mm_D0.9mm_OD2.3mm -> Teapot:PogoPinContact_2_P4.8mm_D2.3mm_H0.7mm
Changed lines of the file:
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@@
   )
   (text "3.3vS = 3.3V for SWARM Satellite Transceiver ( Max 2A )"
-    (at 132.08 81.28 0)
+    (at 132.08 81.28 180)
     (effects (font (size 1.27 1.27)) (justify right bottom))
   )
@@
     (property "Reference" "J4" (id 0) (at 83.82 118.11 0))
     (property "Value" "5V" (id 1) (at 83.82 120.65 0))
-    (property "Footprint" "Connector_Wire:SolderWire-0.5sqmm_1x02_P4.8mm_D0.9mm_OD2.3mm" (id 2) (at 83.82 127 0)
+    (property "Footprint" "Teapot:PogoPinContact_2_P4.8mm_D2.3mm_H0.7mm" (id 2) (at 83.82 127 0)
       (effects (font (size 1.27 1.27)) hide)
     )
@@
     (property "Reference" "J2" (id 0) (at 83.82 54.61 0))
     (property "Value" "3.3V SWARM" (id 1) (at 83.82 57.15 0))
-    (property "Footprint" "Connector_Wire:SolderWire-0.5sqmm_1x02_P4.8mm_D0.9mm_OD2.3mm" (id 2) (at 83.82 63.5 0)
+    (property "Footprint" "Teapot:PogoPinContact_2_P4.8mm_D2.3mm_H0.7mm" (id 2) (at 83.82 63.5 0)
       (effects (font (size 1.27 1.27)) hide)
     )
@@
     (property "Reference" "J1" (id 0) (at 83.82 86.36 0))
     (property "Value" "3.3V LoRaWAN" (id 1) (at 83.82 88.9 0))
-    (property "Footprint" "Connector_Wire:SolderWire-0.5sqmm_1x02_P4.8mm_D0.9mm_OD2.3mm" (id 2) (at 83.82 95.25 0)
+    (property "Footprint" "Teapot:PogoPinContact_2_P4.8mm_D2.3mm_H0.7mm" (id 2) (at 83.82 95.25 0)
       (effects (font (size 1.27 1.27)) hide)
     )
@@
     (property "Reference" "J6" (id 0) (at 181.61 119.38 0))
     (property "Value" "12V" (id 1) (at 181.61 121.92 0))
-    (property "Footprint" "Connector_Wire:SolderWire-0.5sqmm_1x02_P4.8mm_D0.9mm_OD2.3mm" (id 2) (at 181.61 128.27 0)
-      (effects (font (size 1.27 1.27)) hide)
-    )
+    (property "Footprint" "Teapot:PogoPinContact_2_P4.8mm_D2.3mm_H0.7mm" (id 2) (at 181.61 128.27 0)
+      (effects (font (size 1.27 1.27)) hide)
+    )
